Commit message: Derived matrices A, B, C, K, unobservable when solving for L

File: projects/03_spacecraft/urdf/spacecraft.urdf (robot description, URDF)
Before this commit: robot spacecraft, 12 links, 11 joints
Joints:
- joint bus_to_mass_1: origin xyz=0.00000000 -0.00000000 -0.00000000 rpy=0.00000000 0.00000000 0.00000000 -> xyz=0.00000000 -0.00000000 -0.40262794 rpy=0.00000000 0.00000000 0.00000000
- joint bus_to_mass_4: origin xyz=0.00000000 0.00000000 0.00000000 rpy=0.00000000 0.00000000 0.00000000 -> xyz=0.00000002 0.00000000 0.00000002 rpy=0.00000000 0.00000000 0.00000000
- joint bus_to_mass_5: origin xyz=-0.00000000 -0.00000000 -0.00000000 rpy=0.00000000 0.00000000 0.00000000 -> xyz=-0.00000002 -0.00000000 -0.00000002 rpy=0.00000000 0.00000000 0.00000000
- joint bus_to_mass_6: origin xyz=0.00000000 -0.00000001 0.00000001 rpy=0.00000000 0.00000000 0.00000000 -> xyz=0.00000000 0.00000001 0.00000001 rpy=0.00000000 0.00000000 0.00000000
- joint bus_to_mass_7: origin xyz=-0.00000000 0.00000001 -0.00000001 rpy=0.00000000 0.00000000 0.00000000 -> xyz=-0.00000000 -0.00000001 -0.00000001 rpy=0.00000000 0.00000000 0.00000000
- joint bus_to_wheel_1: origin xyz=1.55563492 1.55563492 0.00000000 rpy=1.57079633 0.00000000 2.35619449 -> xyz=1.79629248 0.00000000 1.27017059 rpy=0.95531662 0.00000000 1.57079633
- joint bus_to_wheel_2: origin xyz=-1.55563492 1.55563492 0.00000000 rpy=1.57079633 0.00000000 3.92699082 -> xyz=-0.89814624 1.55563492 1.27017059 rpy=0.95531662 0.00000000 3.66519143
- joint bus_to_wheel_3: origin xyz=-1.55563492 -1.55563492 0.00000000 rpy=1.57079633 0.00000000 5.49778714 -> xyz=-0.89814624 -1.55563492 1.27017059 rpy=0.95531662 0.00000000 5.75958653
- joint bus_to_wheel_4: origin xyz=1.55563492 -1.55563492 0.00000000 rpy=1.57079633 0.00000000 7.06858347 -> xyz=0.00000000 0.00000000 -2.20000000 rpy=3.14159265 0.00000000 1.57079633

Commit message: Created an iteration to loop through different wheel placements, attempt to optimize best wheel placement vs. success rate. Current best success rate 90%.

File: projects/03_spacecraft/urdf/spacecraft.urdf (robot description, URDF)
Before this commit: robot spacecraft, 12 links, 11 joints
Joints:
- joint bus_to_mass_1: origin xyz=0.00000000 -0.00000000 -0.40262794 rpy=0.00000000 0.00000000 0.00000000 -> xyz=-0.13750000 -0.23815699 -0.40262794 rpy=0.00000000 0.00000000 0.00000000
- joint bus_to_mass_2: origin xyz=-0.00000003 0.00000003 0.00000000 rpy=0.00000000 0.00000000 0.00000000 -> xyz=-0.91749864 0.91749864 0.00000000 rpy=0.00000000 0.00000000 0.00000000
- joint bus_to_mass_3: origin xyz=0.00000003 -0.00000003 -0.00000000 rpy=0.00000000 0.00000000 0.00000000 -> xyz=0.91749864 -0.91749864 -0.00000000 rpy=0.00000000 0.00000000 0.00000000
- joint bus_to_mass_4: origin xyz=0.00000002 0.00000000 0.00000002 rpy=0.00000000 0.00000000 0.00000000 -> xyz=0.63782263 0.00000000 0.63782263 rpy=0.00000000 0.00000000 0.00000000
- joint bus_to_mass_5: origin xyz=-0.00000002 -0.00000000 -0.00000002 rpy=0.00000000 0.00000000 0.00000000 -> xyz=-0.63782263 -0.00000000 -0.63782263 rpy=0.00000000 0.00000000 0.00000000
- joint bus_to_mass_6: origin xyz=0.00000000 0.00000001 0.00000001 rpy=0.00000000 0.00000000 0.00000000 -> xyz=0.00000000 0.83942179 0.83942179 rpy=0.00000000 0.00000000 0.00000000
- joint bus_to_mass_7: origin xyz=-0.00000000 -0.00000001 -0.00000001 rpy=0.00000000 0.00000000 0.00000000 -> xyz=-0.00000000 -0.83942179 -0.83942179 rpy=0.00000000 0.00000000 0.00000000
- joint bus_to_wheel_1: origin xyz=1.79629248 0.00000000 1.27017059 rpy=0.95531662 0.00000000 1.57079633 -> xyz=1.10000000 1.90525589 0.00000000 rpy=1.57079633 0.00000000 2.61799388
- joint bus_to_wheel_2: origin xyz=-0.89814624 1.55563492 1.27017059 rpy=0.95531662 0.00000000 3.66519143 -> xyz=-1.10000000 0.00000000 1.90525589 rpy=0.52359878 0.00000000 4.71238898
- joint bus_to_wheel_3: origin xyz=-0.89814624 -1.55563492 1.27017059 rpy=0.95531662 0.00000000 5.75958653 -> xyz=0.55000000 -0.95262794 1.90525589 rpy=0.52359878 0.00000000 6.80678408

Commit message: made potential fixes to iterations file

File: projects/03_spacecraft/urdf/spacecraft.urdf (robot description, URDF)
Before this commit: robot spacecraft, 12 links, 11 joints
Joints:
- joint bus_to_mass_1: origin xyz=-0.13750000 -0.23815699 -0.40262794 rpy=0.00000000 0.00000000 0.00000000 -> xyz=0.00000000 0.00000000 0.34284387 rpy=0.00000000 0.00000000 0.00000000
- joint bus_to_mass_2: origin xyz=-0.91749864 0.91749864 0.00000000 rpy=0.00000000 0.00000000 0.00000000 -> xyz=-0.00000000 0.00000000 0.00000000 rpy=0.00000000 0.00000000 0.00000000
- joint bus_to_mass_3: origin xyz=0.91749864 -0.91749864 -0.00000000 rpy=0.00000000 0.00000000 0.00000000 -> xyz=0.00000000 -0.00000000 -0.00000000 rpy=0.00000000 0.00000000 0.00000000
- joint bus_to_mass_4: origin xyz=0.63782263 0.00000000 0.63782263 rpy=0.00000000 0.00000000 0.00000000 -> xyz=0.00000000 0.00000000 0.00000000 rpy=0.00000000 0.00000000 0.00000000
- joint bus_to_mass_5: origin xyz=-0.63782263 -0.00000000 -0.63782263 rpy=0.00000000 0.00000000 0.00000000 -> xyz=-0.00000000 -0.00000000 -0.00000000 rpy=0.00000000 0.00000000 0.00000000
- joint bus_to_mass_6: origin xyz=0.00000000 0.83942179 0.83942179 rpy=0.00000000 0.00000000 0.00000000 -> xyz=0.00000000 0.00000001 0.00000001 rpy=0.00000000 0.00000000 0.00000000
- joint bus_to_mass_7: origin xyz=-0.00000000 -0.83942179 -0.83942179 rpy=0.00000000 0.00000000 0.00000000 -> xyz=-0.00000000 -0.00000001 -0.00000001 rpy=0.00000000 0.00000000 0.00000000
- joint bus_to_wheel_1: origin xyz=1.10000000 1.90525589 0.00000000 rpy=1.57079633 0.00000000 2.61799388 -> xyz=1.09129614 1.89018036 0.27620817 rpy=1.44491497 0.00000000 2.61799388
- joint bus_to_wheel_2: origin xyz=-1.10000000 0.00000000 1.90525589 rpy=0.52359878 0.00000000 4.71238898 -> xyz=-2.18259228 0.00000000 0.27620817 rpy=1.44491497 0.00000000 4.71238898
- joint bus_to_wheel_3: origin xyz=0.55000000 -0.95262794 1.90525589 rpy=0.52359878 0.00000000 6.80678408 -> xyz=1.09129614 -1.89018036 0.27620817 rpy=1.44491497 0.00000000 6.80678408

Commit message: 94% success rate

File: projects/03_spacecraft/urdf/spacecraft.urdf (robot description, URDF)
Before this commit: robot spacecraft, 12 links, 11 joints
Joints:
- joint bus_to_mass_1: origin xyz=0.00000000 0.00000000 0.34284387 rpy=0.00000000 0.00000000 0.00000000 -> xyz=0.00000000 0.00000000 -0.27500000 rpy=0.00000000 0.00000000 0.00000000
- joint bus_to_mass_2: origin xyz=-0.00000000 0.00000000 0.00000000 rpy=0.00000000 0.00000000 0.00000000 -> xyz=-0.00000003 0.00000003 0.00000000 rpy=0.00000000 0.00000000 0.00000000
- joint bus_to_mass_3: origin xyz=0.00000000 -0.00000000 -0.00000000 rpy=0.00000000 0.00000000 0.00000000 -> xyz=0.00000003 -0.00000003 -0.00000000 rpy=0.00000000 0.00000000 0.00000000
- joint bus_to_mass_4: origin xyz=0.00000000 0.00000000 0.00000000 rpy=0.00000000 0.00000000 0.00000000 -> xyz=-0.00000001 0.00000000 0.00000001 rpy=0.00000000 0.00000000 0.00000000
- joint bus_to_mass_5: origin xyz=-0.00000000 -0.00000000 -0.00000000 rpy=0.00000000 0.00000000 0.00000000 -> xyz=0.00000001 -0.00000000 -0.00000001 rpy=0.00000000 0.00000000 0.00000000
- joint bus_to_mass_6: origin xyz=0.00000000 0.00000001 0.00000001 rpy=0.00000000 0.00000000 0.00000000 -> xyz=0.00000000 0.00000002 0.00000002 rpy=0.00000000 0.00000000 0.00000000
- joint bus_to_mass_7: origin xyz=-0.00000000 -0.00000001 -0.00000001 rpy=0.00000000 0.00000000 0.00000000 -> xyz=-0.00000000 -0.00000002 -0.00000002 rpy=0.00000000 0.00000000 0.00000000
- joint bus_to_wheel_1: origin xyz=1.09129614 1.89018036 0.27620817 rpy=1.44491497 0.00000000 2.61799388 -> xyz=0.95262794 1.65000000 1.10000000 rpy=1.04719755 0.00000000 2.61799388
- joint bus_to_wheel_2: origin xyz=-2.18259228 0.00000000 0.27620817 rpy=1.44491497 0.00000000 4.71238898 -> xyz=-1.90525589 0.00000000 1.10000000 rpy=1.04719755 0.00000000 4.71238898
- joint bus_to_wheel_3: origin xyz=1.09129614 -1.89018036 0.27620817 rpy=1.44491497 0.00000000 6.80678408 -> xyz=0.95262794 -1.65000000 1.10000000 rpy=1.04719755 0.00000000 6.80678408

Commit message: Successfully collected data from iterations of different wheel placements vs. success rate. Best experimental delta value = 0.44 (96% success rate). Best theoretical delta value = 0.54 (94% success rate)

File: projects/03_spacecraft/urdf/spacecraft.urdf (robot description, URDF)
Before this commit: robot spacecraft, 12 links, 11 joints
Joints:
- joint bus_to_mass_1: origin xyz=0.00000000 0.00000000 -0.27500000 rpy=0.00000000 0.00000000 0.00000000 -> xyz=0.00000000 0.00000000 -0.89041652 rpy=0.00000000 0.00000000 0.00000000
- joint bus_to_mass_2: origin xyz=-0.00000003 0.00000003 0.00000000 rpy=0.00000000 0.00000000 0.00000000 -> xyz=-0.00000001 0.00000001 0.00000000 rpy=0.00000000 0.00000000 0.00000000
- joint bus_to_mass_3: origin xyz=0.00000003 -0.00000003 -0.00000000 rpy=0.00000000 0.00000000 0.00000000 -> xyz=0.00000001 -0.00000001 -0.00000000 rpy=0.00000000 0.00000000 0.00000000
- joint bus_to_mass_4: origin xyz=-0.00000001 0.00000000 0.00000001 rpy=0.00000000 0.00000000 0.00000000 -> xyz=0.00000003 0.00000000 0.00000003 rpy=0.00000000 0.00000000 0.00000000
- joint bus_to_mass_5: origin xyz=0.00000001 -0.00000000 -0.00000001 rpy=0.00000000 0.00000000 0.00000000 -> xyz=-0.00000003 -0.00000000 -0.00000003 rpy=0.00000000 0.00000000 0.00000000
- joint bus_to_mass_6: origin xyz=0.00000000 0.00000002 0.00000002 rpy=0.00000000 0.00000000 0.00000000 -> xyz=0.00000000 0.00000003 0.00000003 rpy=0.00000000 0.00000000 0.00000000
- joint bus_to_mass_7: origin xyz=-0.00000000 -0.00000002 -0.00000002 rpy=0.00000000 0.00000000 0.00000000 -> xyz=-0.00000000 -0.00000003 -0.00000003 rpy=0.00000000 0.00000000 0.00000000
- joint bus_to_wheel_1: origin xyz=0.95262794 1.65000000 1.10000000 rpy=1.04719755 0.00000000 2.61799388 -> xyz=0.53653217 0.92930098 1.92055537 rpy=0.50951799 0.00000000 2.61799388
- joint bus_to_wheel_2: origin xyz=-1.90525589 0.00000000 1.10000000 rpy=1.04719755 0.00000000 4.71238898 -> xyz=-1.07306435 0.00000000 1.92055537 rpy=0.50951799 0.00000000 4.71238898
- joint bus_to_wheel_3: origin xyz=0.95262794 -1.65000000 1.10000000 rpy=1.04719755 0.00000000 6.80678408 -> xyz=0.53653217 -0.92930098 1.92055537 rpy=0.50951799 0.00000000 6.80678408

Commit message: 97% success rate, r=0.2 for stars

File: projects/03_spacecraft/urdf/spacecraft.urdf (robot description, URDF)
Before this commit: robot spacecraft, 12 links, 11 joints
Joints:
- joint bus_to_mass_1: origin xyz=0.00000000 0.00000000 -0.89041652 rpy=0.00000000 0.00000000 0.00000000 -> xyz=0.00000000 0.00000000 0.00991072 rpy=0.00000000 0.00000000 0.00000000
- joint bus_to_mass_4: origin xyz=0.00000003 0.00000000 0.00000003 rpy=0.00000000 0.00000000 0.00000000 -> xyz=0.00000002 0.00000000 0.00000002 rpy=0.00000000 0.00000000 0.00000000
- joint bus_to_mass_5: origin xyz=-0.00000003 -0.00000000 -0.00000003 rpy=0.00000000 0.00000000 0.00000000 -> xyz=-0.00000002 -0.00000000 -0.00000002 rpy=0.00000000 0.00000000 0.00000000
- joint bus_to_wheel_1: origin xyz=0.53653217 0.92930098 1.92055537 rpy=0.50951799 0.00000000 2.61799388 -> xyz=1.03940230 1.80029759 0.72011904 rpy=1.23732315 0.00000000 2.61799388
- joint bus_to_wheel_2: origin xyz=-1.07306435 0.00000000 1.92055537 rpy=0.50951799 0.00000000 4.71238898 -> xyz=-2.07880460 0.00000000 0.72011904 rpy=1.23732315 0.00000000 4.71238898
- joint bus_to_wheel_3: origin xyz=0.53653217 -0.92930098 1.92055537 rpy=0.50951799 0.00000000 6.80678408 -> xyz=1.03940230 -1.80029759 0.72011904 rpy=1.23732315 0.00000000 6.80678408
